Commit message: 修复头部相机坐标系

File: src/robot_description/urdf/camera_optical_link.xacro (robot description, xacro)
@@ -2,4 +2,21 @@
 <robot xmlns:xacro="http://www.ros.org/wiki/xacro">
   <xacro:macro name="camera_optical_link">
+    <!-- 头部相机 -->
+    <link name="head_camera_optical_link">
+      <collision>
+        <origin xyz="0 0 0.0001" rpy="0 0 0"/>
+        <geometry>
+          <box size="0.0001 0.0001 0.0001"/>
+        </geometry>
+      </collision>
+    </link>
+    <joint
+      name="head_camera_optical_joint"
+      type="fixed">
+      <parent link="head_camera_link"/>
+      <child link="head_camera_optical_link"/>
+      <origin xyz="0 0 0" rpy="-1.57079632679 0.0 -1.57079632679"/>
+    </joint>
+    <!-- 右手相机 -->
     <link name="right_camera_optical_link">
       <collision>
@@ -16,4 +33,5 @@
       <origin xyz="0 0 0" rpy="0 1.57079632679 0"/>
     </joint>
+    <!-- 左手相机 -->
     <link name="left_camera_optical_link">
       <collision>

File: src/robot_description/urdf/humanoid.gazebo.xacro (robot description, xacro)
@@ -8,5 +8,5 @@
     </gazebo>
     <!-- 头部深度相机（RGB-D） -->
-    <gazebo reference="head_camera_link">
+    <gazebo reference="head_camera_optical_link">
       <sensor name="head_camera" type="rgbd_camera">
         <pose>0 0 0 0 -1.5708 1.5708</pose>
